File: pcb/MGC_module.kicad_pcb (KiCad board)
At the start: 2 copper layers, 33 x 48.9 mm, 48 parts, among them J11 103P012BB100, J12 103P012BB100, J13 103P012BB100, J3 103P012BB100, J7 103P012BB100, SW1 SW_DIP_x02, U1 DG418LDY, U2 DG418LDY, U3 ATmega4809-A, Y1 32.768k

Commit message: Fix pwm value/routing issue
Parts:
- R10: value 150 -> 10k
- R13, R14: value 22k -> 0R
- R15: renamed from R16; value 0 -> 0R
- R16: renamed from R15; value 0 -> 0R
- R4, R5: value 0 -> 0R
Connections:
- R16 pad 1: /PD2 -> /PD4
Routing:
- net /PD2: track 29.9 -> 25.2 mm, vias 3 -> 2
- net /PD4: track 19.5 -> 22.0 mm
Changed lines of the file:
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@@
 			)
 		)
-		(property "Value" "0"
+		(property "Value" "0R"
 			(at 0 1.524 90)
 			(layer "B.Fab")
@@
 		(descr "Resistor SMD 1206 (3216 Metric), square (rectangular) end terminal, IPC-7351 nominal, (Body size source: IPC-SM-782 page 72, https://www.pcb-3d.com/wordpress/wp-content/uploads/ipc-sm-782a_amendment_1_and_2.pdf), generated with kicad-footprint-generator")
 		(tags "resistor")
-		(property "Reference" "R15"
+		(property "Reference" "R16"
 			(at 3.048 0 90)
 			(layer "B.SilkS")
@@
 			)
 		)
-		(property "Value" "0"
+		(property "Value" "0R"
 			(at 0 -1.651 90)
 			(layer "B.Fab")
@@
 			(layers "B.Cu" "B.Mask" "B.Paste")
 			(roundrect_rratio 0.222222)
-			(net 35 "/PD2")
+			(net 33 "/PD4")
 			(pintype "passive")
 		)
@@
 			)
 		)
-		(property "Value" "150"
+		(property "Value" "10k"
 			(at 0 -1.651 90)
 			(layer "B.Fab")
@@
 			)
 		)
-		(property "HTL" "102934"
+		(property "HTL" "102967"
 			(at 0 0 90)
 			(unlocked yes)
@@
 			)
 		)
-		(property "Value" "22k"
+		(property "Value" "0R"
 			(at 0 1.778 0)
 			(layer "B.Fab")
@@
 			)
 		)
-		(property "HTL" "102934"
+		(property "HTL" "102902"
 			(at 0 0 180)
 			(unlocked yes)
@@
 			)
 		)
-		(property "Value" "0"
+		(property "Value" "0R"
 			(at 0 -1.651 90)
 			(layer "B.Fab")
@@
 			)
 		)
-		(property "Value" "22k"
+		(property "Value" "0R"
 			(at 0 -1.651 0)
 			(layer "B.Fab")
@@
 			)
 		)
-		(property "HTL" "102934"
+		(property "HTL" "102902"
 			(at 0 0 180)
 			(unlocked yes)
@@
 		(descr "Resistor SMD 1206 (3216 Metric), square (rectangular) end terminal, IPC-7351 nominal, (Body size source: IPC-SM-782 page 72, https://www.pcb-3d.com/wordpress/wp-content/uploads/ipc-sm-782a_amendment_1_and_2.pdf), generated with kicad-footprint-generator")
 		(tags "resistor")
-		(property "Reference" "R16"
+		(property "Reference" "R15"
 			(at 3.048 0.381 90)
 			(layer "B.SilkS")
@@
 			)
 		)
-		(property "Value" "0"
+		(property "Value" "0R"
 			(at 0 -1.651 90)
 			(layer "B.Fab")
@@
 	(segment
 		(start 134.493 92.964001)
+		(end 137.795 92.964001)
+		(width 0.18)
+		(layer "B.Cu")
+		(net 33)
+	)
+	(segment
+		(start 137.795 92.964001)
+		(end 136.525 92.964001)
+		(width 0.18)
+		(layer "B.Cu")
+		(net 33)
+	)
+	(segment
+		(start 136.525 92.964001)
+		(end 136.398 92.837001)
+		(width 0.18)
+		(layer "B.Cu")
+		(net 33)
+	)
+	(segment
+		(start 137.795 92.964001)
 		(end 140.208 92.964001)
 		(width 0.18)
@@
 	)
 	(segment
+		(start 136.398 92.837001)
+		(end 136.398 91.755501)
+		(width 0.18)
+		(layer "B.Cu")
+		(net 33)
+	)
+	(segment
 		(start 138.811 87.630001)
 		(end 135.255 87.630001)
@@
 	)
 	(via
-		(at 139.319 89.027001)
-		(size 0.4)
-		(drill 0.3)
-		(layers "F.Cu" "B.Cu")
-		(net 35)
-	)
-	(via
 		(at 149.832 91.440001)
 		(size 0.4)
@@
 	)
 	(segment
-		(start 139.319 90.170001)
-		(end 139.319 89.027001)
-		(width 0.18)
-		(layer "B.Cu")
-		(net 35)
-	)
-	(segment
-		(start 136.398 91.755501)
-		(end 137.7335 91.755501)
-		(width 0.18)
-		(layer "B.Cu")
-		(net 35)
-	)
-	(segment
 		(start 149.832 91.440001)
 		(end 149.832 94.389501)
 		(width 0.18)
 		(layer "B.Cu")
-		(net 35)
-	)
-	(segment
-		(start 137.7335 91.755501)
-		(end 139.319 90.170001)
-		(width 0.18)
-		(layer "B.Cu")
