File: pcb/MGC_module.kicad_sch (KiCad schematic)
At the start: 47 parts, among them J11 103P012BB100, J12 103P012BB100, J13 103P012BB100, J3 103P012BB100, J7 103P012BB100, SW1 SW_DIP_x02, U1 DG418LDY, U2 DG418LDY, U3 ATmega4809-A, Y1 32.768k

Commit message: Fix pwm value/routing issue
Parts:
- R10: value 150 -> 10k; HTL 102934 -> 102967
- R13, R14: value 22k -> 0R; HTL 102934 -> 102902
- R15: renamed from R16; value 0 -> 0R
- R16: renamed from R15; value 0 -> 0R
- R4, R5: value 0 -> 0R
Connections:
- net PD2: no longer R16.1
- net PD4: now also R16.1
Other:
- moved on the sheet: R16
Changed lines of the file:
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@@
 	(wire
 		(pts
-			(xy 118.11 135.89) (xy 118.11 140.97)
-		)
-		(stroke
-			(width 0)
-			(type default)
-		)
-	)
-	(wire
-		(pts
 			(xy 180.34 38.1) (xy 180.34 31.75)
 		)
@@
 	(wire
 		(pts
-			(xy 113.03 135.89) (xy 113.03 144.78)
+			(xy 113.03 135.89) (xy 113.03 140.97)
 		)
 		(stroke
@@
 	(wire
 		(pts
-			(xy 113.03 152.4) (xy 113.03 153.67)
+			(xy 118.11 152.4) (xy 118.11 157.48)
 		)
 		(stroke
@@
 	(wire
 		(pts
-			(xy 115.57 152.4) (xy 115.57 153.67)
+			(xy 115.57 152.4) (xy 115.57 157.48)
 		)
 		(stroke
@@
 	(wire
 		(pts
+			(xy 118.11 135.89) (xy 118.11 144.78)
+		)
+		(stroke
+			(width 0)
+			(type default)
+		)
+	)
+	(wire
+		(pts
 			(xy 69.85 105.41) (xy 69.85 100.33)
 		)
@@
 	(global_label "V_POT"
 		(shape output)
-		(at 115.57 153.67 270)
+		(at 115.57 157.48 270)
 		(fields_autoplaced yes)
 		(effects
@@
 		)
 		(property "Intersheetrefs" "${INTERSHEET_REFS}"
-			(at 115.57 162.2795 90)
+			(at 115.57 166.0895 90)
 			(effects
 				(font
@@
 	(global_label "RPM"
 		(shape output)
-		(at 113.03 153.67 270)
+		(at 118.11 157.48 270)
 		(fields_autoplaced yes)
 		(effects
@@
 		)
 		(property "Intersheetrefs" "${INTERSHEET_REFS}"
-			(at 113.03 160.6466 90)
+			(at 118.11 164.4566 90)
 			(effects
 				(font
@@
 		(on_board yes)
 		(dnp no)
-		(property "Reference" "R16"
-			(at 118.11 148.59 90)
+		(property "Reference" "R15"
+			(at 114.3 153.67 90)
 			(effects
 				(font
@@
 			)
 		)
-		(property "Value" "0"
-			(at 114.3 144.78 90)
+		(property "Value" "0R"
+			(at 114.3 143.51 90)
 			(effects
 				(font
@@
 			(project "MGC_module"
 				(path "/74660cec-7259-46bd-b267-6a3b6b13872e"
-					(reference "R16")
+					(reference "R15")
 					(unit 1)
 				)
@@
 			)
 		)
-		(property "Value" "22k"
+		(property "Value" "0R"
 			(at 81.28 143.51 90)
 			(effects
@@
 			)
 		)
-		(property "HTL" "102934"
+		(property "HTL" "102902"
 			(at 82.55 148.59 90)
 			(effects
@@
 			)
 		)
-		(property "Value" "22k"
+		(property "Value" "0R"
 			(at 83.82 143.51 90)
 			(effects
@@
 			)
 		)
-		(property "HTL" "102934"
+		(property "HTL" "102902"
 			(at 85.09 148.59 90)
 			(effects
@@
 			)
 		)
-		(property "Value" "0"
-			(at 114.3 87.63 90)
+		(property "Value" "0R"
+			(at 111.76 87.63 90)
 			(effects
 				(font
@@
 			)
 		)
-		(property "Value" "0"
-			(at 116.84 87.63 90)
+		(property "Value" "0R"
+			(at 114.3 87.63 90)
 			(effects
 				(font
@@
 			)
 		)
-		(property "Value" "150"
+		(property "Value" "10k"
 			(at 177.8 123.19 90)
 			(effects
@@
 			)
 		)
-		(property "HTL" "102934"
+		(property "HTL" "102967"
 			(at 177.8 120.65 90)
 			(effects
@@
 	(symbol
 		(lib_id "Device:R")
-		(at 113.03 148.59 0)
+		(at 118.11 148.59 0)
 		(unit 1)
 		(exclude_from_sim no)
@@
 		(on_board yes)
 		(dnp no)
-		(property "Reference" "R15"
-			(at 110.49 148.59 90)
+		(property "Reference" "R16"
+			(at 116.84 153.67 90)
 			(effects
 				(font
@@
 			)
 		)
-		(property "Value" "0"
-			(at 111.76 144.78 90)
+		(property "Value" "0R"
+			(at 116.84 143.51 90)
 			(effects
 				(font
@@
 		)
 		(property "Footprint" "Resistor_SMD:R_1206_3216Metric"
-			(at 111.252 148.59 90)
+			(at 116.332 148.59 90)
 			(effects
 				(font
@@
 		)
 		(property "Datasheet" "~"
-			(at 113.03 148.59 0)
+			(at 118.11 148.59 0)
 			(effects
 				(font
@@
 		)
 		(property "Description" "Resistor"
-			(at 113.03 148.59 0)
+			(at 118.11 148.59 0)
 			(effects
 				(font
@@
 		)
 		(property "HTL" "102934"
-			(at 113.03 148.59 90)
+			(at 118.11 148.59 90)
 			(effects
 				(font
@@
 		)
 		(property "Sim.Device" ""
-			(at 113.03 148.59 90)
+			(at 118.11 148.59 90)
 			(effects
 				(font
@@
 		)
 		(property "KLC_S3.3" ""
-			(at 113.03 148.59 90)
+			(at 118.11 148.59 90)
 			(effects
 				(font
@@
 		)
 		(property "KLC_S4.1" ""
-			(at 113.03 148.59 90)
+			(at 118.11 148.59 90)
 			(effects
 				(font
@@
 		)
 		(property "Sim.Pins" ""
-			(at 113.03 148.59 90)
+			(at 118.11 148.59 90)
 			(effects
 				(font
@@
 			(project "MGC_module"
 				(path "/74660cec-7259-46bd-b267-6a3b6b13872e"
-					(reference "R15")
+					(reference "R16")
 					(unit 1)
 				)
